File: boards/squishy.sch (KiCad schematic (older format))
At the start: 161 parts, among them J1 USB3_Micro_B_Amphenol, J2 Conn_02x26_Top_Bottom, U1 FT600Q-B-T, U10 THVD1451, U11 THVD1451, U12 THVD1451, U13 THVD1451, U14 THVD1451, U15 THVD1451, U16 THVD1451, U17 THVD1451, U18 THVD1451, U19 THVD1451, U2 ICE40HX8K-BG121, U20 THVD1451, U21 TXB0106, U22 TXB0106, U23 TXB0106, U24 TXB0106, U25 TXB0106, U26 TXB0106, U3 THVD1451, U4 THVD1451, U5 THVD1451, U6 THVD1451, U7 THVD1451, U8 THVD1451, U9 THVD1451

Commit message: Updates, moved to an FTDI chip
Parts:
- removed J1: USB3_Micro_B_Amphenol, lethalbit:USB3_Micro_B_Amphenol, symbol lethalbit:USB3_Micro_B_Amphenol
- removed U1: FT600Q-B-T, lethalbit:QFN-56_EP_7x7_Pitch0.4mm, symbol lethalbit:FT600Q-B-T
- added C35, C36: 47pf, Capacitor_SMD:C_0402_1005Metric, symbol Device:C_Small
- added C37, C38, C39, C40, C42: 0.1uF, Capacitor_SMD:C_0402_1005Metric, symbol Device:C_Small
- added C41: 100uF, Capacitor_SMD:C_1210_3225Metric, symbol Device:C_Small
- added C43: 0.01uF, Capacitor_SMD:C_0402_1005Metric, symbol Device:C_Small
- added J1: USB_B_Micro, lethalbit-connectors:MICRO-USB-B-(IN_PCB), symbol Connector:USB_B_Micro
- added J3: Conn_02x05_Odd_Even, lethalbit-connectors:FTSH-105-01-L-DV-K-TR, symbol Connector_Generic:Conn_02x05_Odd_Even
- added U1: 128MiB, lethalbit-memory:WSON-8-1EP-6.0x8.0mm, symbol lethalbit-memory:W25N01GVZEIG
- added U27: FT240XQ, Package_DFN_QFN:QFN-24-1EP_4x4mm_P0.5mm_EP2.6x2.6mm, symbol Interface_USB:FT240XQ
- added X1: ASEM-48MHz, Oscillator:Oscillator_SMD_Abracon_ASE-4Pin_3.2x2.5mm, symbol Oscillator:ASE-xxxMHz
- C3: value 0.1uF -> 0.01uF; MPN C0402C104M8PACTU -> C0402C103K3RACTU
Connections:
- net labels added: +1V2, +3V3, ACK_RX, ACK_TX, ATN_RX, ATN_TX, BNK0_OE, BNK1_OE, BNK2_OE, BNK3_OE, BNK4_OE, BNK5_OE, BSY_RX, BSY_TX, CD_RX, CD_TX, D+, D-, D0, D1, D2, D3, D4, D5, D6, D7, DB0_RX, DB0_TX, DB1_RX, DB1_TX, DB2_RX, DB2_TX, DB3_RX, DB3_TX, DB4_RX, DB4_TX, DB5_RX, DB5_TX, DB6_RX, DB6_TX, DB7_RX, DB7_TX, DBP_RX, DBP_TX, D[0..7], GLOBAL_CLK, IO_RX, IO_TX, MSG_RX, MSG_TX, REQ_RX, REQ_TX, RST_RX, RST_TX, SEL_RX, SEL_TX, ~RD, ~RXF, ~SI_WU, ~TXF, ~WR
- net labels removed: +3.3V, _0+, _0-, _1+, _1-, _2+, _2-
- wire segments 944 -> 1034
- no-connect marks 1 -> 2
Other:
- moved on the sheet: C1, R1, U2A, U2D

Commit message: Routed the rest of the buses for the level shifters, added the bypass caps, and a whole bunch of other stuff
Parts:
- added C44, C45: 0.1uF, Capacitor_SMD:C_0603_1608Metric, symbol Device:C_Small
- added C46, C47, C48, C49, C50, C51, C52, C53: 0.1uF, Capacitor_SMD:C_0402_1005Metric, symbol Device:C_Small
- added D1, D10, D9: BLUE, LED_SMD:LED_0603_1608Metric_Pad1.05x0.95mm_HandSolder, symbol Device:LED_Small
- added D2, D6: PINK, LED_SMD:LED_0603_1608Metric_Pad1.05x0.95mm_HandSolder, symbol Device:LED_Small
- added D5: WHITE, LED_SMD:LED_0603_1608Metric_Pad1.05x0.95mm_HandSolder, symbol Device:LED_Small
- added R63, R67, R69: 4k7, Resistor_SMD:R_0603_1608Metric, symbol Device:R_Small
- added R64, R66: 10k, Resistor_SMD:R_0603_1608Metric, symbol Device:R_Small
- added R65: 6k8, Resistor_SMD:R_0603_1608Metric, symbol Device:R_Small
- added R68: 100k, Resistor_SMD:R_0603_1608Metric, symbol Device:R_Small
Connections:
- net +1V2: now also C45.2, C47.2, C49.2, C51.2, C53.2
- net +3V3: now also J3.2 (Pin_2), C44.2, C46.2, C48.2, C50.2, C52.2
- net ACK_RX: now also U2.A6 (IOT_206); no longer U2.A9 (IOT_178)
- net ACK_TX: now also U2.B7 (IOT_197_GBIN1); no longer U2.C8 (IOT_179)
- net ATN_RX: now also U2.C4 (IOL_4A); no longer U2.B3 (IOT_221)
- net ATN_TX: now also U2.B3 (IOT_221); no longer U2.A2 (IOT_222)
- net BNK0_OE: now also U2.A1 (IOT_225); no longer U2.A4 (IOT_211)
- net BNK1_OE: now also U2.A4 (IOT_211); no longer U2.A11 (IOT_168)
- net BNK2_OE: now also U2.D7 (IOT_181); no longer U2.G10 (IOR_120)
- net BNK3_OE: now also U2.A11 (IOT_168); no longer U2.B11 (IOR_161)
- net BNK4_OE: now also U2.D11 (IOR_152); no longer U2.E9 (IOR_144)
- net BNK5_OE: now also U2.G9 (IOR_128); no longer U2.C7 (IOT_191)
- net BSY_RX: now also U2.D5 (IOT_212); no longer U2.A10 (IOT_170)
- net BSY_TX: now also U2.B5 (IOT_208); no longer U2.C9 (IOT_172)
- net CD_RX: now also U2.E11 (IOR_148); no longer U2.F9 (IOR_137)
- net CD_TX: now also U2.E10 (IOR_141_GBIN2); no longer U2.F10 (IOR_136)
- net DB0_RX: now also U2.C3 (IOL_4B); no longer U2.D5 (IOT_212)
- net DB0_TX: now also U2.A2 (IOT_222); no longer U2.B4 (IOT_219)
- net DB1_TX: now also U2.B4 (IOT_219); no longer U2.A1 (IOT_225)
- net DB2_RX: now also U2.A5 (IOT_207); no longer U2.B9 (IOT_174)
- net DB2_TX: now also U2.B6 (IOT_198_GBIN0); no longer U2.B8 (IOT_177)
- net DB3_RX: now also U2.C7 (IOT_191); no longer U2.H11 (IOR_119)
- net DB3_TX: now also U2.A7 (IOT_192); no longer U2.G8 (IOR_118)
- net DB4_RX: now also U2.A8 (IOT_190); no longer U2.K11 (IOR_115)
- net DB4_TX: now also U2.C9 (IOT_172); no longer U2.J11 (IOR_114)
- net DB5_RX: now also U2.D9 (IOR_147); no longer U2.D11 (IOR_152)
- net DB5_TX: now also U2.C11 (IOR_160); no longer U2.E11 (IOR_148)
- net DB6_RX: now also U2.D10 (IOR_154); no longer U2.E10 (IOR_141_GBIN2)
- net DB6_TX: now also U2.F9 (IOR_137); no longer U2.F11 (IOR_140_GBIN3)
- net DB7_RX: now also U2.F11 (IOR_140_GBIN3); no longer U2.G11 (IOR_129)
- net DB7_TX: now also U2.F10 (IOR_136); no longer U2.G9 (IOR_128)
- net DBP_RX: now also U2.H11 (IOR_119); no longer U2.B6 (IOT_198_GBIN0)
- net DBP_TX: now also U2.H10 (IOR_116); no longer U2.A6 (IOT_206)
- net GND: now also J3.7 (Pin_7), C44.1, C45.1, C46.1, C47.1, C48.1, C49.1, C50.1, C51.1, C52.1, C53.1, D1.1 (K), D10.1 (K), D2.1 (K), D5.1 (K), D6.1 (K), D9.1 (K), R68.1
- net IO_RX: now also U2.J11 (IOR_114); no longer U2.A5 (IOT_207)
- net IO_TX: now also U2.J10 (IOR_117); no longer U2.B5 (IOT_208)
- net MSG_RX: now also U2.A10 (IOT_170); no longer U2.C11 (IOR_160)
- net MSG_TX: now also U2.B11 (IOR_161); no longer U2.D10 (IOR_154)
- net REQ_RX: now also U2.G11 (IOR_129); no longer U2.A7 (IOT_192)
- net REQ_TX: now also U2.G10 (IOR_120); no longer U2.B7 (IOT_197_GBIN1)
- net RST_RX: now also U2.C8 (IOT_179); no longer U2.J10 (IOR_117)
- net RST_TX: now also U2.B8 (IOT_177); no longer U2.H10 (IOR_116)
- net SEL_RX: now also U2.E8 (IOR_146); no longer U2.D9 (IOR_147)
- net SEL_TX: now also U2.E9 (IOR_144); no longer U2.E8 (IOR_146)
- net FPGA_DONE: now reaches U2.K8 (CDONE)
- net FPGA_DONE: now also R69.1
- net S4: now reaches U2.L1 (IOB_56)
- net S4: now also R66.1
- net S5: now reaches U2.L2 (IOB_61)
- net S5: now also R67.1
- net ~FPGA_RESET: now reaches U2.L9 (~CRESET)
- net ~FPGA_RESET: now also R68.2
- net S1: now reaches U2.H1 (IOL_18A)
- net S1: now also R63.1
- net S2: now reaches U2.J1 (IOL_23A)
- net S2: now also R64.1
- net S3: now reaches U2.K1 (IOL_23B)
- net S3: now also R65.1
- net at U1.2 (DO/IO1), U2.J9 (IOB_106_SDI): now also J3.3 (Pin_3)
- net at U1.1 (~CS), U2.K10 (IOB_108_SS): now also J3.1 (Pin_1)
- net at U1.5 (DI/IO0), U2.K9 (IOB_105_SDO): now also J3.8 (Pin_8)
- net at U1.6 (CLK), U2.L10 (IOB_107_SCK): now also J3.6 (Pin_6)
- net at J3.4 (Pin_4): now also U1.7 (~HOLD~/IO3)
- net at J3.5 (Pin_5): now also U1.3 (~WP~/IO2)
- new net: D1.2 (A), R63.2
- new net: D2.2 (A), R64.2
- new net: D5.2 (A), R65.2
- new net: D9.2 (A), R67.2
- new net: D6.2 (A), R66.2
- new net: D10.2 (A), R69.2
- no-connect marks 2 -> 3
Other:
- moved on the sheet: C23, C24, C25, C26, C27, C28, C29, C30, C31, C32, C33, C34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

Commit message: Completed the routing and power, the last two things to do are sort the SCSI TERMPOWER and DIFFSENSE, and then the FPGA reset.
Parts:
- added C? (x4): 4.7uF, Capacitor_SMD:C_0603_1608Metric, symbol Device:C_Small
- added U?: TLV755533PDRVR, Package_DFN_QFN:DFN-6-1EP_2x2mm_P0.65mm_EP1x1.6mm, symbol lethalbit:TLV755533PDRVR
- added U?: TLV73312PQDRVRQ1, Package_DFN_QFN:DFN-6-1EP_2x2mm_P0.65mm_EP1x1.6mm, symbol lethalbit:TLV73312PQDRVRQ1
- added U?: MAX809JTRG, Package_TO_SOT_SMD:SOT-23, symbol lethalbit:MAX809JTRG
- C44, C45: value 0.1uF -> 4.7uF
Connections:
- net +1V2: now also C?.2, U?.1 (OUT), U?.2 (N2)
- net +3V3: now also C?.2, U?.1 (OUT), U?.2 (N2)
- net +5V: now also C?.2, C?.2, U?.3 (VCC), U?.4 (EN), U?.5 (NC), U?.5 (NC), U?.6 (IN), U?.6 (IN)
- net GND: now also C?.1, C?.1, C?.1, C?.1, U?.1 (GND), U?.3 (GND), U?.3 (GND), U?.7 (GND), U?.7 (GND)
- new net: U?.2 (~RESET), U?.4 (EN)
Other:
- moved on the sheet: C37, C38, C39, C40, U27

Commit message: Added the needed bits for TERMPOWER and for the DIFFSENS line
Parts:
- added F1: Polyfuse_Small, Fuse:Fuse_1210_3225Metric_Castellated, symbol Device:Polyfuse_Small
- added JP1: TERMPWR, Connector_PinHeader_2.54mm:PinHeader_1x02_P2.54mm_Vertical, symbol Device:Jumper_NO_Small
- added R70: 10k, Resistor_SMD:R_0603_1608Metric, symbol Device:R_Small
- gave numbers to parts that had none: 7
Connections:
- net +5V: now also JP1.1; no longer R12.2, R15.2, R18.2, R21.2, R24.2, R27.2, R30.2, R33.2, R36.2, R39.2, R42.2, R45.2, R48.2, R51.2, R54.2, R57.2, R60.2, R9.2
- net DIFF_SENSE: now also R70.1
- net TERMPWR: now also R12.2, R15.2, R18.2, R21.2, R24.2, R27.2, R30.2, R33.2, R36.2, R39.2, R42.2, R45.2, R48.2, R51.2, R54.2, R57.2, R60.2, R9.2, F1.1, R70.2
- net ~FPGA_RESET: now also J3.10 (Pin_10)
- new net: F1.2, JP1.2
Other:
- moved on the sheet: C54, C55, C56, C57, U28, U29, U30

Commit message: Updates to the schematic, REV0 is "done"
Parts:
- added FID1, FID2, FID3, FID4, FID5, FID6: Fiducial, Fiducial:Fiducial_0.75mm_Mask1.5mm, symbol Mechanical:Fiducial
- added R71: 10k, Resistor_SMD:R_0603_1608Metric, symbol Device:R_Small
- added TP1: 1v2, TestPoint:TestPoint_Pad_D1.0mm, symbol Connector:TestPoint_Small
- added TP2: 5v0, TestPoint:TestPoint_Pad_D1.0mm, symbol Connector:TestPoint_Small
- added TP3: 3v3, TestPoint:TestPoint_Pad_D1.0mm, symbol Connector:TestPoint_Small
- added TP4: GND, TestPoint:TestPoint_Pad_D1.0mm, symbol Connector:TestPoint_Small
- R68: value 100k -> 10k; MPN CRCW0603100KFKEA -> CRCW060310K0FKEA
Connections:
- net +1V2: now also TP1.1
- net +3V3: now also R68.2, R71.2, TP3.1
- net +5V: now also TP2.1
- net DIFF_SENSE: now also U2.A9 (IOT_178)
- net GND: now also TP4.1; no longer R68.1
- net ~FPGA_RESET: now also R68.1; no longer R68.2
- net at J3.1 (Pin_1), U1.1 (~CS), U2.K10 (IOB_108_SS): now also R71.1
Changed lines of the file:
@@
 U 1 1 5F40EB64
 P 15450 4700
-F 0 "C42" V 15600 4550 50  0000 C CNN
-F 1 "0.1uF" V 15600 4750 50  0000 C CNN
+F 0 "C42" V 15350 4700 50  0000 C CNN
+F 1 "0.1uF" V 15550 4700 50  0000 C CNN
 F 2 "Capacitor_SMD:C_0402_1005Metric" H 15450 4700 50  0001 C CNN
 F 3 "~" H 15450 4700 50  0001 C CNN
@@
 Text Label 4450 14500 2    50   ~ 0
 ~SI_WU
-NoConn ~ 20850 11950
 NoConn ~ 20850 12050
 Wire Wire Line
@@
 Wire Wire Line
 	15850 6700 15850 7000
-$Comp
-L power:GND #PWR0203
-U 1 1 773AACDB
-P 10300 6050
-F 0 "#PWR0203" H 10300 5800 50  0001 C CNN
-F 1 "GND" H 10305 5877 50  0000 C CNN
-F 2 "" H 10300 6050 50  0001 C CNN
-F 3 "" H 10300 6050 50  0001 C CNN
-	1    10300 6050
-	1    0    0    -1
-$EndComp
-Wire Wire Line
-	10300 5950 10300 6050
-$Comp
-L Device:R_Small R68
-U 1 1 77A76F0B
-P 10300 5850
-F 0 "R68" V 10104 5850 50  0000 C CNN
-F 1 "100k" V 10195 5850 50  0000 C CNN
-F 2 "Resistor_SMD:R_0603_1608Metric" H 10300 5850 50  0001 C CNN
-F 3 "~" H 10300 5850 50  0001 C CNN
-F 4 "Vishay Dale" V 10300 5850 50  0001 C CNN "MFR"
-F 5 "CRCW0603100KFKEA" V 10300 5850 50  0001 C CNN "MPN"
-	1    10300 5850
-	-1   0    0    1
-$EndComp
 Wire Wire Line
 	10900 5700 10300 5700
 Wire Wire Line
-	10300 5700 10300 5750
-Text Label 10300 5700 0    50   ~ 0
+	10300 5700 10300 5550
+Text Label 10350 5700 0    50   ~ 0
 ~FPGA_RESET
 Wire Wire Line
@@
 Wire Wire Line
 	18700 6850 18700 7300
+Connection ~ 18700 7300
+Wire Wire Line
+	18700 7300 18400 7300
+$Comp
+L Connector:TestPoint_Small TP1
+U 1 1 81852B35
+P 2300 7000
+F 0 "TP1" H 2348 7046 50  0000 L CNN
+F 1 "1v2" H 2348 6955 50  0000 L CNN
+F 2 "TestPoint:TestPoint_Pad_D1.0mm" H 2500 7000 50  0001 C CNN
+F 3 "~" H 2500 7000 50  0001 C CNN
+	1    2300 7000
+	1    0    0    -1
+$EndComp
+$Comp
+L Connector:TestPoint_Small TP2
+U 1 1 81856755
+P 2300 7200
+F 0 "TP2" H 2348 7246 50  0000 L CNN
+F 1 "5v0" H 2348 7155 50  0000 L CNN
+F 2 "TestPoint:TestPoint_Pad_D1.0mm" H 2500 7200 50  0001 C CNN
+F 3 "~" H 2500 7200 50  0001 C CNN
+	1    2300 7200
+	1    0    0    -1
+$EndComp
+$Comp
+L Connector:TestPoint_Small TP3
+U 1 1 819F814A
+P 2300 7400
+F 0 "TP3" H 2348 7446 50  0000 L CNN
+F 1 "3v3" H 2348 7355 50  0000 L CNN
+F 2 "TestPoint:TestPoint_Pad_D1.0mm" H 2500 7400 50  0001 C CNN
+F 3 "~" H 2500 7400 50  0001 C CNN
+	1    2300 7400
+	1    0    0    -1
+$EndComp
+$Comp
+L Connector:TestPoint_Small TP4
+U 1 1 819F8150
+P 2300 7600
+F 0 "TP4" H 2348 7646 50  0000 L CNN
+F 1 "GND" H 2348 7555 50  0000 L CNN
+F 2 "TestPoint:TestPoint_Pad_D1.0mm" H 2500 7600 50  0001 C CNN
+F 3 "~" H 2500 7600 50  0001 C CNN
+	1    2300 7600
+	1    0    0    -1
+$EndComp
+Wire Wire Line
+	2200 7000 2200 6950
+$Comp
+L power:+1V2 #PWR0150
+U 1 1 81B9B76B
+P 2200 6950
+F 0 "#PWR0150" H 2200 6800 50  0001 C CNN
+F 1 "+1V2" H 2215 7123 50  0000 C CNN
+F 2 "" H 2200 6950 50  0001 C CNN
+F 3 "" H 2200 6950 50  0001 C CNN
+	1    2200 6950
+	1    0    0    -1
+$EndComp
+Wire Wire Line
+	2200 7000 2300 7000
+$Comp
+L power:+5V #PWR0154
+U 1 1 81EE6EFC
+P 2000 6950
+F 0 "#PWR0154" H 2000 6800 50  0001 C CNN
+F 1 "+5V" H 2015 7123 50  0000 C CNN
+F 2 "" H 2000 6950 50  0001 C CNN
+F 3 "" H 2000 6950 50  0001 C CNN
+	1    2000 6950
+	1    0    0    -1
+$EndComp
+Wire Wire Line
+	2000 7200 2300 7200
+Wire Wire Line
+	2000 6950 2000 7200
+$Comp
+L power:+3V3 #PWR0156
+U 1 1 82580D3A
+P 1800 6950
+F 0 "#PWR0156" H 1800 6800 50  0001 C CNN
+F 1 "+3V3" H 1815 7123 50  0000 C CNN
+F 2 "" H 1800 6950 50  0001 C CNN
+F 3 "" H 1800 6950 50  0001 C CNN
+	1    1800 6950
+	1    0    0    -1
+$EndComp
+Wire Wire Line
+	1800 7400 2300 7400
+Wire Wire Line
+	1800 6950 1800 7400
+$Comp
+L power:GND #PWR0158
+U 1 1 828D1004
+P 1800 8000
+F 0 "#PWR0158" H 1800 7750 50  0001 C CNN
+F 1 "GND" H 1805 7827 50  0000 C CNN
+F 2 "" H 1800 8000 50  0001 C CNN
+F 3 "" H 1800 8000 50  0001 C CNN
+	1    1800 8000
+	1    0    0    -1
+$EndComp
+Wire Wire Line
+	1800 8000 1800 7600
+Wire Wire Line
+	1800 7600 2300 7600
+$Comp
+L Device:R_Small R71
+U 1 1 835EE3E5
+P 15650 5100
+F 0 "R71" V 15454 5100 50  0000 C CNN
+F 1 "10k" V 15545 5100 50  0000 C CNN
+F 2 "Resistor_SMD:R_0603_1608Metric" H 15650 5100 50  0001 C CNN
+F 3 "~" H 15650 5100 50  0001 C CNN
+F 4 "Vishay Dale" V 15650 5100 50  0001 C CNN "MFR"
+F 5 "CRCW060310K0FKEA" V 15650 5100 50  0001 C CNN "MPN"
+	1    15650 5100
+	-1   0    0    1
+$EndComp
+Wire Wire Line
+	15650 5650 15650 5200
+Connection ~ 15650 5650
+Wire Wire Line
+	15650 5000 15650 4550
+Wire Wire Line
+	15650 4550 15450 4550
+Connection ~ 15450 4550
+NoConn ~ 20850 11950
+$Comp
+L Device:R_Small R68
+U 1 1 83CEA5CA
+P 10300 5450
+F 0 "R68" V 10104 5450 50  0000 C CNN
+F 1 "10k" V 10195 5450 50  0000 C CNN
+F 2 "Resistor_SMD:R_0603_1608Metric" H 10300 5450 50  0001 C CNN
+F 3 "~" H 10300 5450 50  0001 C CNN
+F 4 "Vishay Dale" V 10300 5450 50  0001 C CNN "MFR"
+F 5 "CRCW060310K0FKEA" V 10300 5450 50  0001 C CNN "MPN"
+	1    10300 5450
+	-1   0    0    1
+$EndComp
+Wire Wire Line
+	10300 5250 10300 5350
+$Comp
+L power:+3V3 #PWR0160
+U 1 1 841EEDDB
+P 10300 5250
+F 0 "#PWR0160" H 10300 5100 50  0001 C CNN
+F 1 "+3V3" H 10315 5423 50  0000 C CNN
+F 2 "" H 10300 5250 50  0001 C CNN
+F 3 "" H 10300 5250 50  0001 C CNN
+	1    10300 5250
+	1    0    0    -1
+$EndComp
+Text Label 2000 14000 2    50   ~ 0
+DIFF_SENSE
+Wire Wire Line
+	1600 14000 2000 14000
+$Comp
+L Mechanical:Fiducial FID1
+U 1 1 849D26AC
+P 2300 8200
+F 0 "FID1" H 2385 8246 50  0000 L CNN
+F 1 "Fiducial" H 2385 8155 50  0000 L CNN
+F 2 "Fiducial:Fiducial_0.75mm_Mask1.5mm" H 2300 8200 50  0001 C CNN
+F 3 "~" H 2300 8200 50  0001 C CNN
+	1    2300 8200
+	1    0    0    -1
+$EndComp
+$Comp
+L Mechanical:Fiducial FID2
+U 1 1 849DA2D2
+P 2300 8400
+F 0 "FID2" H 2385 8446 50  0000 L CNN
+F 1 "Fiducial" H 2385 8355 50  0000 L CNN
+F 2 "Fiducial:Fiducial_0.75mm_Mask1.5mm" H 2300 8400 50  0001 C CNN
+F 3 "~" H 2300 8400 50  0001 C CNN
+	1    2300 8400
+	1    0    0    -1
+$EndComp
+$Comp
+L Mechanical:Fiducial FID3
+U 1 1 849DA4BA
+P 2300 8600
+F 0 "FID3" H 2385 8646 50  0000 L CNN
+F 1 "Fiducial" H 2385 8555 50  0000 L CNN
+F 2 "Fiducial:Fiducial_0.75mm_Mask1.5mm" H 2300 8600 50  0001 C CNN
+F 3 "~" H 2300 8600 50  0001 C CNN
+	1    2300 8600
+	1    0    0    -1
+$EndComp
+$Comp
+L Mechanical:Fiducial FID4
+U 1 1 849E7F8A
+P 2800 8200
+F 0 "FID4" H 2885 8246 50  0000 L CNN
+F 1 "Fiducial" H 2885 8155 50  0000 L CNN
+F 2 "Fiducial:Fiducial_0.75mm_Mask1.5mm" H 2800 8200 50  0001 C CNN
+F 3 "~" H 2800 8200 50  0001 C CNN
+	1    2800 8200
+	1    0    0    -1
+$EndComp
+$Comp
+L Mechanical:Fiducial FID5
+U 1 1 849E7F90
+P 2800 8400
+F 0 "FID5" H 2885 8446 50  0000 L CNN
+F 1 "Fiducial" H 2885 8355 50  0000 L CNN
+F 2 "Fiducial:Fiducial_0.75mm_Mask1.5mm" H 2800 8400 50  0001 C CNN
+F 3 "~" H 2800 8400 50  0001 C CNN
+	1    2800 8400
+	1    0    0    -1
+$EndComp
+$Comp
+L Mechanical:Fiducial FID6
+U 1 1 849E7F96
+P 2800 8600
+F 0 "FID6" H 2885 8646 50  0000 L CNN
+F 1 "Fiducial" H 2885 8555 50  0000 L CNN
+F 2 "Fiducial:Fiducial_0.75mm_Mask1.5mm" H 2800 8600 50  0001 C CNN
+F 3 "~" H 2800 8600 50  0001 C CNN
+	1    2800 8600
+	1    0    0    -1
+$EndComp
 Wire Bus Line
 	21100 10550 21100 11250
 Wire Bus Line
 	4800 13300 4800 14300
-Connection ~ 18700 7300
-Wire Wire Line
-	18700 7300 18400 7300
 $EndSCHEMATC

Commit message: Fixed some part attributes
Parts:
- U2: MFR (none) -> Lattice Semicondutors; MPN (none) -> ICE40HX8K-BG121
- U2: MFR (none) -> Lattice Semiconductors; MPN (none) -> ICE40HX8K-BG121
- U2: MFR (none) -> Lattice Semiconducrtors; MPN (none) -> ICE40HX8K-BG121
- X1: FPN ASEMB-48.000MHZ-LY-T -> (none); MPN (none) -> ASEMB-48.000MHZ-LY-T
Changed lines of the file:
@@
 F 2 "Package_BGA:BGA-121_9.0x9.0mm_Layout11x11_P0.8mm_Ball0.4mm_Pad0.35mm_NSMD" H 2400 12950 50  0001 C CNN
 F 3 "http://www.latticesemi.com/Products/FPGAandCPLD/iCE40" H 1550 15400 50  0001 C CNN
+F 4 "Lattice Semicondutors" H 2400 14400 50  0001 C CNN "MFR"
+F 5 "ICE40HX8K-BG121" H 2400 14400 50  0001 C CNN "MPN"
 	2    2400 14400
 	-1   0    0    -1
@@
 F 2 "Package_BGA:BGA-121_9.0x9.0mm_Layout11x11_P0.8mm_Ball0.4mm_Pad0.35mm_NSMD" H 1100 12850 50  0001 C CNN
 F 3 "http://www.latticesemi.com/Products/FPGAandCPLD/iCE40" H 250 15300 50  0001 C CNN
+F 4 "Lattice Semiconductors" H 1100 14300 50  0001 C CNN "MFR"
+F 5 "ICE40HX8K-BG121" H 1100 14300 50  0001 C CNN "MPN"
 	1    1100 14300
 	-1   0    0    -1
@@
 F 2 "Package_BGA:BGA-121_9.0x9.0mm_Layout11x11_P0.8mm_Ball0.4mm_Pad0.35mm_NSMD" H 11500 5250 50  0001 C CNN
 F 3 "http://www.latticesemi.com/Products/FPGAandCPLD/iCE40" H 10650 7700 50  0001 C CNN
+F 4 "Lattice Semiconductors" H 11500 6700 50  0001 C CNN "MFR"
+F 5 "ICE40HX8K-BG121" H 11500 6700 50  0001 C CNN "MPN"
 	3    11500 6700
 	1    0    0    -1
@@
 F 2 "Package_BGA:BGA-121_9.0x9.0mm_Layout11x11_P0.8mm_Ball0.4mm_Pad0.35mm_NSMD" H 3700 12850 50  0001 C CNN
 F 3 "http://www.latticesemi.com/Products/FPGAandCPLD/iCE40" H 2850 15300 50  0001 C CNN
+F 4 "Lattice Semiconducrtors" H 3700 14300 50  0001 C CNN "MFR"
+F 5 "ICE40HX8K-BG121" H 3700 14300 50  0001 C CNN "MPN"
 	4    3700 14300
 	-1   0    0    -1
@@
 F 2 "Package_BGA:BGA-121_9.0x9.0mm_Layout11x11_P0.8mm_Ball0.4mm_Pad0.35mm_NSMD" H 14850 4000 50  0001 C CNN
 F 3 "http://www.latticesemi.com/Products/FPGAandCPLD/iCE40" H 14000 6450 50  0001 C CNN
+F 4 "Lattice Semiconductors" H 14850 5450 50  0001 C CNN "MFR"
+F 5 "ICE40HX8K-BG121" H 14850 5450 50  0001 C CNN "MPN"
 	5    14850 5450
 	-1   0    0    -1
@@
 F 3 "http://abracon.com/Oscillators/ASEMB.pdf" H 20000 13850 50  0001 C CNN
 F 4 "Abracon" H 20100 13850 50  0001 C CNN "MFR"
-F 5 "ASEMB-48.000MHZ-LY-T" H 20100 13850 50  0001 C CNN "FPN"
+F 5 "ASEMB-48.000MHZ-LY-T" H 20100 13850 50  0001 C CNN "MPN"
 	1    20100 13850
 	1    0    0    -1
