File: rev0/kicad-proj/squishy.sch (KiCad schematic (older format))
At the start: 217 parts, among them J1 USB_B_Micro, J2 Conn_02x26_Top_Bottom, J3 Conn_02x05_Odd_Even, U1 128MiB, U10 THVD1451, U11 THVD1451, U12 THVD1451, U13 THVD1451, U14 THVD1451, U15 THVD1451, U16 THVD1451, U17 THVD1451, U18 THVD1451, U19 THVD1451, U2 ICE40HX8K-BG121, U20 THVD1451, U21 TXB0106, U22 TXB0106, U23 TXB0106, U24 TXB0106, U25 TXB0106, U26 TXB0106, U27 FT240XQ, U28 MAX809JTRG, U29 TLV755533PDRVR, U3 THVD1451, U30 TLV73312PQDRVRQ1, U4 THVD1451, U5 THVD1451, U6 THVD1451, U7 THVD1451, U8 THVD1451, U9 THVD1451, X1 ASEM-48MHz

Commit message: Moved some things around and cached the rev0 of squishy
Parts:
- J1: symbol squishy-rescue:USB_B_Micro-Connector -> Connector:USB_B_Micro
Changed lines of the file:
@@
 	16150 14400 15950 14400
 $Comp
-L squishy-rescue:USB_B_Micro-Connector J1
+L Connector:USB_B_Micro J1
 U 1 1 70E3C85C
 P 900 1550

Commit message: hardware: massive board overhaul for rev1
Parts:
- J1: symbol Connector:USB_B_Micro -> squishy-rescue:USB_B_Micro-Connector
Changed lines of the file:
@@
 Wire Wire Line
 	20600 7150 20600 7500
-Text Label 19300 5050 0    50   ~ 0
-DB0+
-Text Label 19300 5150 0    50   ~ 0
-DB0-
-Text Label 19300 5250 0    50   ~ 0
-DB1+
-Text Label 19300 5350 0    50   ~ 0
-DB1-
-Text Label 19300 5450 0    50   ~ 0
-DB2+
-Text Label 19300 5550 0    50   ~ 0
-DB2-
-Text Label 19300 5650 0    50   ~ 0
-DB3+
-Text Label 19300 5750 0    50   ~ 0
-DB3-
-Text Label 19300 5850 0    50   ~ 0
-DB4+
-Text Label 19300 5950 0    50   ~ 0
-DB4-
-Text Label 19300 6050 0    50   ~ 0
-DB5+
-Text Label 19300 6150 0    50   ~ 0
-DB5-
-Text Label 19300 6250 0    50   ~ 0
-DB6+
-Text Label 19300 6350 0    50   ~ 0
-DB6-
-Text Label 19300 6450 0    50   ~ 0
-DB7+
-Text Label 19300 6550 0    50   ~ 0
-DB7-
-Text Label 19300 6650 0    50   ~ 0
-DBP+
-Text Label 19300 6750 0    50   ~ 0
-DBP-
 Text Label 19300 6850 0    50   ~ 0
 DIFF_SENSE
@@
 Text Label 19300 7350 0    50   ~ 0
 TERMPWR
-Text Label 20400 5050 2    50   ~ 0
-ATN+
-Text Label 20400 5150 2    50   ~ 0
-ATN-
-Text Label 20400 5450 2    50   ~ 0
-BSY+
-Text Label 20400 5550 2    50   ~ 0
-BSY-
-Text Label 20400 5650 2    50   ~ 0
-ACK+
-Text Label 20400 5750 2    50   ~ 0
-ACK-
-Text Label 20400 5850 2    50   ~ 0
-RST+
-Text Label 20400 5950 2    50   ~ 0
-RST-
-Text Label 20400 6050 2    50   ~ 0
-MSG+
-Text Label 20400 6150 2    50   ~ 0
-MSG-
-Text Label 20400 6250 2    50   ~ 0
-SEL+
-Text Label 20400 6350 2    50   ~ 0
-SEL-
-Text Label 20400 6450 2    50   ~ 0
-CD+
-Text Label 20400 6550 2    50   ~ 0
-CD-
-Text Label 20400 6650 2    50   ~ 0
-REQ+
-Text Label 20400 6750 2    50   ~ 0
-REQ-
-Text Label 20400 6850 2    50   ~ 0
-IO+
-Text Label 20400 6950 2    50   ~ 0
-IO-
 $Comp
 L lethalbit:THVD1451 U4
@@
 	16150 14400 15950 14400
 $Comp
-L Connector:USB_B_Micro J1
+L squishy-rescue:USB_B_Micro-Connector J1
 U 1 1 70E3C85C
 P 900 1550
@@
 Wire Bus Line
 	4800 13300 4800 14300
+Text Label 19300 6650 0    50   ~ 0
+DBP+
+Text Label 19300 6750 0    50   ~ 0
+DBP-
+Text Label 19300 5050 0    50   ~ 0
+DB0+
+Text Label 19300 5150 0    50   ~ 0
+DB0-
+Text Label 19300 5250 0    50   ~ 0
+DB1+
+Text Label 19300 5350 0    50   ~ 0
+DB1-
+Text Label 19300 5450 0    50   ~ 0
+DB2+
+Text Label 19300 5550 0    50   ~ 0
+DB2-
+Text Label 19300 5650 0    50   ~ 0
+DB3+
+Text Label 19300 5750 0    50   ~ 0
+DB3-
+Text Label 19300 5850 0    50   ~ 0
+DB4+
+Text Label 19300 5950 0    50   ~ 0
+DB4-
+Text Label 19300 6050 0    50   ~ 0
+DB5+
+Text Label 19300 6150 0    50   ~ 0
+DB5-
+Text Label 19300 6250 0    50   ~ 0
+DB6+
+Text Label 19300 6350 0    50   ~ 0
+DB6-
+Text Label 19300 6450 0    50   ~ 0
+DB7+
+Text Label 19300 6550 0    50   ~ 0
+DB7-
+Text Label 20400 6950 2    50   ~ 0
+IO-
+Text Label 20400 6850 2    50   ~ 0
+IO+
+Text Label 20400 6550 2    50   ~ 0
+CD-
+Text Label 20400 6450 2    50   ~ 0
+CD+
+Text Label 20400 5750 2    50   ~ 0
+ACK-
+Text Label 20400 5650 2    50   ~ 0
+ACK+
+Text Label 20400 6350 2    50   ~ 0
+SEL-
+Text Label 20400 6250 2    50   ~ 0
+SEL+
+Text Label 20400 5150 2    50   ~ 0
+ATN-
+Text Label 20400 5050 2    50   ~ 0
+ATN+
+Text Label 20400 5550 2    50   ~ 0
+BSY-
+Text Label 20400 5450 2    50   ~ 0
+BSY+
+Text Label 20400 6150 2    50   ~ 0
+MSG-
+Text Label 20400 6050 2    50   ~ 0
+MSG+
+Text Label 20400 6750 2    50   ~ 0
+REQ-
+Text Label 20400 6650 2    50   ~ 0
+REQ+
+Text Label 20400 5950 2    50   ~ 0
+RST-
+Text Label 20400 5850 2    50   ~ 0
+RST+
 $EndSCHEMATC
