File: boards/squishy/squishy-mechanical.kicad_sch (KiCad schematic)
At the start: 12 parts

Commit message: hardware: cleanup and revamp for squishy rev2
Parts:
- G2: renamed from G1; value Graphic -> Ran-Filled
- H1, H2, H3, H4: footprint MountingHole:MountingHole_3.2mm_M3 -> MountingHole:MountingHole_3.2mm_M3_Pad
- renumbered FID2 to FID1, FID5 to FID2, FID1 to FID5, G2 to G1
Other:
- note added: "Fiducials"
- note added: "Graphics"
- note added: "Mounting Holes"
- title: (none) -> Squishy
- moved on the sheet: FID1, FID2, FID3, FID4, FID5, FID6, G2, H1

Commit message: hardware: lots of work on the initial layout of rev2, not gonnya but too much effort in now though until we find all the problems with rev1
Parts:
- H1, H2, H3, H4: symbol Mechanical:MountingHole -> Mechanical:MountingHole_Pad
Connections:
- new net GND: H1.1, H2.1, H3.1, H4.1
Changed lines of the file:
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@@
     (comment 1 "Mechanical")
+  )
+  (junction (at 67.31 26.67) (diameter 0) (color 0 0 0 0))
+  (junction (at 67.31 36.83) (diameter 0) (color 0 0 0 0))
+  (wire (pts (xy 62.23 26.67) (xy 67.31 26.67))
+    (stroke (width 0) (type default) (color 0 0 0 0))
+  )
+  (wire (pts (xy 67.31 26.67) (xy 72.39 26.67))
+    (stroke (width 0) (type default) (color 0 0 0 0))
+  )
+  (wire (pts (xy 67.31 36.83) (xy 62.23 36.83))
+    (stroke (width 0) (type default) (color 0 0 0 0))
+  )
+  (wire (pts (xy 67.31 36.83) (xy 67.31 26.67))
+    (stroke (width 0) (type default) (color 0 0 0 0))
+  )
+  (wire (pts (xy 67.31 38.1) (xy 67.31 36.83))
+    (stroke (width 0) (type default) (color 0 0 0 0))
+  )
+  (wire (pts (xy 72.39 36.83) (xy 67.31 36.83))
+    (stroke (width 0) (type default) (color 0 0 0 0))
   )
   (polyline (pts (xy 13.97 13.97) (xy 13.97 41.91))
@@
     (effects (font (size 1.27 1.27)) (justify left bottom))
   )
+  (symbol (lib_id "power:GND") (at 67.31 38.1 0) (unit 1)
+    (in_bom yes) (on_board yes)
+    (property "Reference" "#PWR0105" (id 0) (at 67.31 44.45 0)
+      (effects (font (size 1.27 1.27)) hide)
+    )
+    (property "Value" "GND" (id 1) (at 71.12 40.64 0))
+    (property "Footprint" "" (id 2) (at 67.31 38.1 0)
+      (effects (font (size 1.27 1.27)) hide)
+    )
+    (property "Datasheet" "" (id 3) (at 67.31 38.1 0)
+      (effects (font (size 1.27 1.27)) hide)
+    )
+    (pin "1")
+  )
   (symbol (lib_id "Mechanical:Fiducial") (at 17.78 21.59 0) (unit 1)
     (in_bom yes) (on_board yes)
@@
     )
   )
-  (symbol (lib_id "Mechanical:MountingHole") (at 59.69 24.13 0) (unit 1)
-    (in_bom yes) (on_board yes)
-    (property "Reference" "H1" (id 0) (at 59.69 19.05 0))
-    (property "Value" "MountingHole" (id 1) (at 59.69 20.955 0))
-    (property "Footprint" "MountingHole:MountingHole_3.2mm_M3_Pad" (id 2) (at 59.69 24.13 0)
-      (effects (font (size 1.27 1.27)) hide)
-    )
-    (property "Datasheet" "~" (id 3) (at 59.69 24.13 0)
-      (effects (font (size 1.27 1.27)) hide)
-    )
-    (property "MFR" "N/A" (id 4) (at 59.69 24.13 0)
-      (effects (font (size 1.27 1.27)) hide)
-    )
-    (property "MPN" "N/A" (id 5) (at 59.69 24.13 0)
-      (effects (font (size 1.27 1.27)) hide)
-    )
-  )
-  (symbol (lib_id "Mechanical:MountingHole") (at 59.69 35.56 0) (unit 1)
-    (in_bom yes) (on_board yes)
-    (property "Reference" "H3" (id 0) (at 59.69 30.48 0))
-    (property "Value" "MountingHole" (id 1) (at 59.69 32.385 0))
-    (property "Footprint" "MountingHole:MountingHole_3.2mm_M3_Pad" (id 2) (at 59.69 35.56 0)
-      (effects (font (size 1.27 1.27)) hide)
-    )
-    (property "Datasheet" "~" (id 3) (at 59.69 35.56 0)
-      (effects (font (size 1.27 1.27)) hide)
-    )
-    (property "MFR" "N/A" (id 4) (at 59.69 35.56 0)
-      (effects (font (size 1.27 1.27)) hide)
-    )
-    (property "MPN" "N/A" (id 5) (at 59.69 35.56 0)
-      (effects (font (size 1.27 1.27)) hide)
-    )
-  )
-  (symbol (lib_id "Mechanical:MountingHole") (at 74.93 24.13 0) (unit 1)
-    (in_bom yes) (on_board yes)
-    (property "Reference" "H2" (id 0) (at 74.93 19.05 0))
-    (property "Value" "MountingHole" (id 1) (at 74.93 20.955 0))
-    (property "Footprint" "MountingHole:MountingHole_3.2mm_M3_Pad" (id 2) (at 74.93 24.13 0)
-      (effects (font (size 1.27 1.27)) hide)
-    )
-    (property "Datasheet" "~" (id 3) (at 74.93 24.13 0)
-      (effects (font (size 1.27 1.27)) hide)
-    )
-    (property "MFR" "N/A" (id 4) (at 74.93 24.13 0)
-      (effects (font (size 1.27 1.27)) hide)
-    )
-    (property "MPN" "N/A" (id 5) (at 74.93 24.13 0)
-      (effects (font (size 1.27 1.27)) hide)
-    )
-  )
-  (symbol (lib_id "Mechanical:MountingHole") (at 74.93 35.56 0) (unit 1)
-    (in_bom yes) (on_board yes)
-    (property "Reference" "H4" (id 0) (at 74.93 30.48 0))
-    (property "Value" "MountingHole" (id 1) (at 74.93 32.385 0))
-    (property "Footprint" "MountingHole:MountingHole_3.2mm_M3_Pad" (id 2) (at 74.93 35.56 0)
-      (effects (font (size 1.27 1.27)) hide)
-    )
-    (property "Datasheet" "~" (id 3) (at 74.93 35.56 0)
-      (effects (font (size 1.27 1.27)) hide)
-    )
-    (property "MFR" "N/A" (id 4) (at 74.93 35.56 0)
-      (effects (font (size 1.27 1.27)) hide)
-    )
-    (property "MPN" "N/A" (id 5) (at 74.93 35.56 0)
-      (effects (font (size 1.27 1.27)) hide)
-    )
+  (symbol (lib_id "Mechanical:MountingHole_Pad") (at 59.69 26.67 90) (unit 1)
+    (in_bom yes) (on_board yes)
+    (property "Reference" "H1" (id 0) (at 58.42 20.32 90))
+    (property "Value" "MountingHole" (id 1) (at 57.785 22.86 90))
+    (property "Footprint" "MountingHole:MountingHole_3.2mm_M3_Pad" (id 2) (at 59.69 26.67 0)
+      (effects (font (size 1.27 1.27)) hide)
+    )
+    (property "Datasheet" "~" (id 3) (at 59.69 26.67 0)
+      (effects (font (size 1.27 1.27)) hide)
+    )
+    (property "MFR" "N/A" (id 4) (at 59.69 26.67 0)
+      (effects (font (size 1.27 1.27)) hide)
+    )
+    (property "MPN" "N/A" (id 5) (at 59.69 26.67 0)
+      (effects (font (size 1.27 1.27)) hide)
+    )
+    (pin "1")
+  )
+  (symbol (lib_id "Mechanical:MountingHole_Pad") (at 59.69 36.83 90) (unit 1)
+    (in_bom yes) (on_board yes)
+    (property "Reference" "H3" (id 0) (at 58.42 30.48 90))
+    (property "Value" "MountingHole" (id 1) (at 59.055 33.02 90))
+    (property "Footprint" "MountingHole:MountingHole_3.2mm_M3_Pad" (id 2) (at 59.69 36.83 0)
+      (effects (font (size 1.27 1.27)) hide)
+    )
+    (property "Datasheet" "~" (id 3) (at 59.69 36.83 0)
+      (effects (font (size 1.27 1.27)) hide)
+    )
+    (property "MFR" "N/A" (id 4) (at 59.69 36.83 0)
+      (effects (font (size 1.27 1.27)) hide)
+    )
+    (property "MPN" "N/A" (id 5) (at 59.69 36.83 0)
+      (effects (font (size 1.27 1.27)) hide)
+    )
+    (pin "1")
+  )
+  (symbol (lib_id "Mechanical:MountingHole_Pad") (at 74.93 26.67 270) (unit 1)
+    (in_bom yes) (on_board yes)
+    (property "Reference" "H2" (id 0) (at 76.2 20.32 90))
+    (property "Value" "MountingHole" (id 1) (at 76.835 22.86 90))
+    (property "Footprint" "MountingHole:MountingHole_3.2mm_M3_Pad" (id 2) (at 74.93 26.67 0)
+      (effects (font (size 1.27 1.27)) hide)
+    )
+    (property "Datasheet" "~" (id 3) (at 74.93 26.67 0)
+      (effects (font (size 1.27 1.27)) hide)
+    )
+    (property "MFR" "N/A" (id 4) (at 74.93 26.67 0)
+      (effects (font (size 1.27 1.27)) hide)
+    )
+    (property "MPN" "N/A" (id 5) (at 74.93 26.67 0)
+      (effects (font (size 1.27 1.27)) hide)
+    )
+    (pin "1")
+  )
+  (symbol (lib_id "Mechanical:MountingHole_Pad") (at 74.93 36.83 270) (unit 1)
+    (in_bom yes) (on_board yes)
+    (property "Reference" "H4" (id 0) (at 76.2 30.48 90))
+    (property "Value" "MountingHole" (id 1) (at 76.835 33.02 90))
+    (property "Footprint" "MountingHole:MountingHole_3.2mm_M3_Pad" (id 2) (at 74.93 36.83 0)
+      (effects (font (size 1.27 1.27)) hide)
+    )
+    (property "Datasheet" "~" (id 3) (at 74.93 36.83 0)
+      (effects (font (size 1.27 1.27)) hide)
+    )
+    (property "MFR" "N/A" (id 4) (at 74.93 36.83 0)
+      (effects (font (size 1.27 1.27)) hide)
+    )
+    (property "MPN" "N/A" (id 5) (at 74.93 36.83 0)
+      (effects (font (size 1.27 1.27)) hide)
+    )
+    (pin "1")
   )
   (symbol (lib_id "lethalbit-graphics:Graphic") (at 27.94 160.02 0) (unit 1)

Commit message: hardware: some silkscreen adjustments
Parts:
- G2: footprint lethalbit-graphics:ran-filled -> lethalbit-graphics:yuki_10x11
Changed lines of the file:
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@@
     (property "Reference" "G2" (id 0) (at 27.94 156.21 0))
     (property "Value" "Ran-Filled" (id 1) (at 27.94 163.83 0))
-    (property "Footprint" "lethalbit-graphics:ran-filled" (id 2) (at 27.94 160.02 0)
+    (property "Footprint" "lethalbit-graphics:yuki_10x11" (id 2) (at 27.94 160.02 0)
       (effects (font (size 1.27 1.27)) hide)
     )

Commit message: hardware: did a whole lot of work on changing the form factor of the board as well as finally assigning the signals and some initial routing.
Parts:
- G1: footprint lethalbit-graphics:Antifaschistische Aktion_600dpi -> DX-MON:Antifaschistische-Aktion_Inv_600dpi
Changed lines of the file:
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@@
       (effects (font (size 1.27 1.27)) (justify left) hide)
     )
-    (property "Footprint" "lethalbit-graphics:Antifaschistische Aktion_600dpi" (id 2) (at 76.2 43.18 0)
+    (property "Footprint" "DX-MON:Antifaschistische-Aktion_Inv_600dpi" (id 2) (at 76.2 43.18 0)
       (effects (font (size 1.27 1.27)) hide)
     )
