File: boards/scsi-50-tap/scsi-50-tap.kicad_sch (KiCad schematic)
At the start: 27 parts, among them J1 SIDE-A, J2 SIDE-B, J3 TAP-OUT, U1 Capacitive-PCB-Diff-Tap, U10 Capacitive-PCB-Diff-Tap, U11 Capacitive-PCB-Diff-Tap, U12 Capacitive-PCB-Diff-Tap, U13 Capacitive-PCB-Diff-Tap, U14 Capacitive-PCB-Diff-Tap, U15 Capacitive-PCB-Diff-Tap, U16 Capacitive-PCB-Diff-Tap, U17 Capacitive-PCB-Diff-Tap, U2 Capacitive-PCB-Diff-Tap, U3 Capacitive-PCB-Diff-Tap, U4 Capacitive-PCB-Diff-Tap, U5 Capacitive-PCB-Diff-Tap, U6 Capacitive-PCB-Diff-Tap, U7 Capacitive-PCB-Diff-Tap, U8 Capacitive-PCB-Diff-Tap, U9 Capacitive-PCB-Diff-Tap

Commit message: hardware: scsi-tap: 50: Updated the 50-pin scsi tap, still needs some work
Parts:
- removed U1, U10, U11, U12, U13, U14, U15, U16, U17, U2, U3, U4, U5, U6, U7, U8, U9, ~1: Capacitive-PCB-Diff-Tap, symbol lethalbit:Capacitive-PCB-Diff-Tap
- added C10, C11, C12, C13, C14, C15, C16, C17, C18, C19, C20, C21, C22, C23, C24, C25, C26, C27, C28, C29, C30, C31, C32, C33, C34, C35, C36, C37, C38, C39, C4, C5, C6, C7, C8, C9: 16pF, Capacitor_SMD:C_0402_1005Metric, symbol Device:C_Small
Connections:
- net SCSI-B.ACK+ is gone; now on net SCSI-P.ACK+: J2.18 (Pin_18)
- net SCSI-B.ACK- is gone; now on net SCSI-P.ACK-: J2.43 (Pin_43)
- net SCSI-B.ATN+ is gone; now on net SCSI-P.ATN+: J2.15 (Pin_15)
- net SCSI-B.ATN- is gone; now on net SCSI-P.ATN-: J2.40 (Pin_40)
- net SCSI-B.BSY+ is gone; now on net SCSI-P.BSY+: J2.17 (Pin_17)
- net SCSI-B.BSY- is gone; now on net SCSI-P.BSY-: J2.42 (Pin_42)
- net SCSI-B.CD+ is gone; now on net SCSI-P.CD+: J2.22 (Pin_22)
- net SCSI-B.CD- is gone; now on net SCSI-P.CD-: J2.47 (Pin_47)
- net SCSI-B.DB0+ is gone; now on net SCSI-P.DB0+: J2.2 (Pin_2)
- net SCSI-B.DB0- is gone; now on net SCSI-P.DB0-: J2.27 (Pin_27)
- net SCSI-B.DB1+ is gone; now on net SCSI-P.DB1+: J2.3 (Pin_3)
- net SCSI-B.DB1- is gone; now on net SCSI-P.DB1-: J2.28 (Pin_28)
- net SCSI-B.DB2+ is gone; now on net SCSI-P.DB2+: J2.4 (Pin_4)
- net SCSI-B.DB2- is gone; now on net SCSI-P.DB2-: J2.29 (Pin_29)
- net SCSI-B.DB3+ is gone; now on net SCSI-P.DB3+: J2.5 (Pin_5)
- net SCSI-B.DB3- is gone; now on net SCSI-P.DB3-: J2.30 (Pin_30)
- net SCSI-B.DB4+ is gone; now on net SCSI-P.DB4+: J2.6 (Pin_6)
- net SCSI-B.DB4- is gone; now on net SCSI-P.DB4-: J2.31 (Pin_31)
- net SCSI-B.DB5+ is gone; now on net SCSI-P.DB5+: J2.7 (Pin_7)
- net SCSI-B.DB5- is gone; now on net SCSI-P.DB5-: J2.32 (Pin_32)
- net SCSI-B.DB6+ is gone; now on net SCSI-P.DB6+: J2.8 (Pin_8)
- net SCSI-B.DB6- is gone; now on net SCSI-P.DB6-: J2.33 (Pin_33)
- net SCSI-B.DB7+ is gone; now on net SCSI-P.DB7+: J2.9 (Pin_9)
- net SCSI-B.DB7- is gone; now on net SCSI-P.DB7-: J2.34 (Pin_34)
- net SCSI-B.DBP+ is gone; now on net SCSI-P.DBP+: J2.10 (Pin_10)
- net SCSI-B.DBP- is gone; now on net SCSI-P.DBP-: J2.35 (Pin_35)
- net SCSI-B.IO+ is gone; now on net SCSI-P.IO+: J2.24 (Pin_24)
- net SCSI-B.IO- is gone; now on net SCSI-P.IO-: J2.49 (Pin_49)
- net SCSI-B.MSG+ is gone; now on net SCSI-P.MSG+: J2.20 (Pin_20)
- net SCSI-B.MSG- is gone; now on net SCSI-P.MSG-: J2.45 (Pin_45)
- net SCSI-B.REQ+ is gone; now on net SCSI-P.REQ+: J2.23 (Pin_23)
- net SCSI-B.REQ- is gone; now on net SCSI-P.REQ-: J2.48 (Pin_48)
- net SCSI-B.RST+ is gone; now on net SCSI-P.RST+: J2.19 (Pin_19)
- net SCSI-B.RST- is gone; now on net SCSI-P.RST-: J2.44 (Pin_44)
- net SCSI-B.SEL+ is gone; now on net SCSI-P.SEL+: J2.21 (Pin_21)
- net SCSI-B.SEL- is gone; now on net SCSI-P.SEL-: J2.46 (Pin_46)
- net SCSI-T.ACK+: now also C26.2
- net SCSI-T.ACK-: now also C27.2
- net SCSI-T.ATN+: now also C22.2
- net SCSI-T.ATN-: now also C23.2
- net SCSI-T.BSY+: now also C24.2
- net SCSI-T.BSY-: now also C25.2
- net SCSI-T.CD+: now also C34.2
- net SCSI-T.CD-: now also C35.2
- net SCSI-T.DB0+: now also C4.2
- net SCSI-T.DB0-: now also C5.2
- net SCSI-T.DB1+: now also C6.2
- net SCSI-T.DB1-: now also C7.2
- net SCSI-T.DB2+: now also C8.2
- net SCSI-T.DB2-: now also C9.2
- net SCSI-T.DB3+: now also C10.2
- net SCSI-T.DB3-: now also C11.2
- net SCSI-T.DB4+: now also C12.2
- net SCSI-T.DB4-: now also C13.2
- net SCSI-T.DB5+: now also C14.2
- net SCSI-T.DB5-: now also C15.2
- net SCSI-T.DB6+: now also C16.2
- net SCSI-T.DB6-: now also C17.2
- net SCSI-T.DB7+: now also C18.2
- net SCSI-T.DB7-: now also C19.2
- net SCSI-T.DBP+: now also C20.2
- net SCSI-T.DBP-: now also C21.2
- net SCSI-T.IO+: now also C38.2
- net SCSI-T.IO-: now also C39.2
- net SCSI-T.MSG+: now also C30.2
- net SCSI-T.MSG-: now also C31.2
- net SCSI-T.REQ+: now also C36.2
- net SCSI-T.REQ-: now also C37.2
- net SCSI-T.RST+: now also C28.2
- net SCSI-T.RST-: now also C29.2
- net SCSI-T.SEL+: now also C32.2
- net SCSI-T.SEL-: now also C33.2
- net SCSI-A.ACK+ renamed SCSI-P.ACK+
- net SCSI-P.ACK+: now also C26.1
- net SCSI-A.ACK- renamed SCSI-P.ACK-
- net SCSI-P.ACK-: now also C27.1
- net SCSI-A.ATN+ renamed SCSI-P.ATN+
- net SCSI-P.ATN+: now also C22.1
- net SCSI-A.ATN- renamed SCSI-P.ATN-
- net SCSI-P.ATN-: now also C23.1
- net SCSI-A.BSY+ renamed SCSI-P.BSY+
- net SCSI-P.BSY+: now also C24.1
- net SCSI-A.BSY- renamed SCSI-P.BSY-
- net SCSI-P.BSY-: now also C25.1
- net SCSI-A.CD+ renamed SCSI-P.CD+
- net SCSI-P.CD+: now also C34.1
- net SCSI-A.CD- renamed SCSI-P.CD-
- net SCSI-P.CD-: now also C35.1
- net SCSI-A.DB0+ renamed SCSI-P.DB0+
- net SCSI-P.DB0+: now also C4.1
- net SCSI-A.DB0- renamed SCSI-P.DB0-
- net SCSI-P.DB0-: now also C5.1
- net SCSI-A.DB1+ renamed SCSI-P.DB1+
- net SCSI-P.DB1+: now also C6.1
- net SCSI-A.DB1- renamed SCSI-P.DB1-
- net SCSI-P.DB1-: now also C7.1
- net SCSI-A.DB2+ renamed SCSI-P.DB2+
- net SCSI-P.DB2+: now also C8.1
- net SCSI-A.DB2- renamed SCSI-P.DB2-
- net SCSI-P.DB2-: now also C9.1
- net SCSI-A.DB3+ renamed SCSI-P.DB3+
- net SCSI-P.DB3+: now also C10.1
- net SCSI-A.DB3- renamed SCSI-P.DB3-
- net SCSI-P.DB3-: now also C11.1
- net SCSI-A.DB4+ renamed SCSI-P.DB4+
- net SCSI-P.DB4+: now also C12.1
- net SCSI-A.DB4- renamed SCSI-P.DB4-
- net SCSI-P.DB4-: now also C13.1
- net SCSI-A.DB5+ renamed SCSI-P.DB5+
- net SCSI-P.DB5+: now also C14.1
- net SCSI-A.DB5- renamed SCSI-P.DB5-
- net SCSI-P.DB5-: now also C15.1
- net SCSI-A.DB6+ renamed SCSI-P.DB6+
- net SCSI-P.DB6+: now also C16.1
- net SCSI-A.DB6- renamed SCSI-P.DB6-
- net SCSI-P.DB6-: now also C17.1
- net SCSI-A.DB7+ renamed SCSI-P.DB7+
- net SCSI-P.DB7+: now also C18.1
- net SCSI-A.DB7- renamed SCSI-P.DB7-
- net SCSI-P.DB7-: now also C19.1
- net SCSI-A.DBP+ renamed SCSI-P.DBP+
- net SCSI-P.DBP+: now also C20.1
- net SCSI-A.DBP- renamed SCSI-P.DBP-
- net SCSI-P.DBP-: now also C21.1
- net SCSI-A.IO+ renamed SCSI-P.IO+
- net SCSI-P.IO+: now also C38.1
- net SCSI-A.IO- renamed SCSI-P.IO-
- net SCSI-P.IO-: now also C39.1
- net SCSI-A.MSG+ renamed SCSI-P.MSG+
- net SCSI-P.MSG+: now also C30.1
- net SCSI-A.MSG- renamed SCSI-P.MSG-
- net SCSI-P.MSG-: now also C31.1
- net SCSI-A.REQ+ renamed SCSI-P.REQ+
- net SCSI-P.REQ+: now also C36.1
- net SCSI-A.REQ- renamed SCSI-P.REQ-
- net SCSI-P.REQ-: now also C37.1
- net SCSI-A.RST+ renamed SCSI-P.RST+
- net SCSI-P.RST+: now also C28.1
- net SCSI-A.RST- renamed SCSI-P.RST-
- net SCSI-P.RST-: now also C29.1
- net SCSI-A.SEL+ renamed SCSI-P.SEL+
- net SCSI-P.SEL+: now also C32.1
- net SCSI-A.SEL- renamed SCSI-P.SEL-
- net SCSI-P.SEL-: now also C33.1
