File: boards/squishy/connector-modules/mse-50-idc/mse-50-idc.kicad_sch (KiCad schematic)
At the start: 12 parts, among them J1 SCSI PHY Mezz, J2 IDC, J3 Conn_01x04, U1 M24C02-RMC

Commit message: squishy: connectors: updated part metadata on mse-50-idc prior to CAM generation
Parts:
- J3: now left out of the parts list
- U1: MFR (none) -> STMicroelectronics; MPN (none) -> M24C02-RMC6TG; SUPPLIER (none) -> DigiKey; SUPPLIER_OC (none) -> 497-17822-1-ND; SUPPLIER_URL (none) -> https://www.digikey.com/short/r9drrzr3
Changed lines of the file:
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@@
 		(unit 1)
 		(exclude_from_sim no)
-		(in_bom yes)
+		(in_bom no)
 		(on_board yes)
 		(dnp no)
@@
 			(at 238.76 147.32 0)
 			(effects
+				(font
+					(size 1.27 1.27)
+				)
+				(hide yes)
+			)
+		)
+		(property "MFR" "STMicroelectronics"
+			(at 238.76 147.32 0)
+			(effects
+				(font
+					(size 1.27 1.27)
+				)
+				(hide yes)
+			)
+		)
+		(property "MPN" "M24C02-RMC6TG"
+			(at 238.76 147.32 0)
+			(effects
+				(font
+					(size 1.27 1.27)
+				)
+				(hide yes)
+			)
+		)
+		(property "SUPPLIER" "DigiKey"
+			(at 238.76 147.32 0)
+			(effects
+				(font
+					(size 1.27 1.27)
+				)
+				(hide yes)
+			)
+		)
+		(property "SUPPLIER_OC" "497-17822-1-ND"
+			(at 238.76 147.32 0)
+			(effects
+				(font
+					(size 1.27 1.27)
+				)
+				(hide yes)
+			)
+		)
+		(property "SUPPLIER_URL" "https://www.digikey.com/short/r9drrzr3"
+			(at 238.76 147.32 0)
+			(effects
